Commit message: Head collision update, weight plugin
Updated the collision of the head to more closely resemble the correct dimensions. Created a plugin to enable adjustable weights to be added to the mouth and tail of the robot, simulating loading or potential tail weights. Hopefully this will allow the trained controller to be able to rapidly respond to changes in the environment

File: frea_description/urdf/frea.urdf.xacro (robot description, xacro)
@@ -27,4 +27,16 @@
         <robotNamespace>/</robotNamespace>
     </plugin>
+    <!-- Plugin to dynamically change the load on the head -->
+    <plugin name="head_weight" filename="libfrea_adjustable_weight.so">
+        <topicName>/adjust_weight/head</topicName>
+        <linkName>head_link</linkName>
+        <position>0.08 0 -0.082</position>
+    </plugin>
+    <!-- Plugin to dynamically change the load on the tail -->
+    <plugin name="tail_weight" filename="libfrea_adjustable_weight.so">
+        <topicName>/adjust_weight/tail</topicName>
+        <linkName>lower_tail_link</linkName>
+        <position>0 0 0.225</position>
+    </plugin>
     <self_collide>false</self_collide>
 </gazebo>

File: frea_description/urdf/head/head.urdf.xacro (robot description, xacro)
@@ -37,7 +37,25 @@
         </visual>
         <collision>
-            <origin xyz="0 0 0" rpy="0 0 0"/>
+            <origin xyz="-0.025 0 0" rpy="0 0 0"/>
             <geometry>
-                <box size="0.134 0.188 0.123"/>
+                <box size="0.15 0.11 0.07"/>
+            </geometry>
+        </collision>
+        <collision>
+            <origin xyz="0.08 0 -0.082" rpy="1.57 0 0"/>
+            <geometry>
+                <cylinder radius="0.003" length="0.065"/>
+            </geometry>
+        </collision>
+        <collision>
+            <origin xyz="0.05 0.035 -0.07" rpy="0 -1.0 0"/>
+            <geometry>
+                <cylinder radius="0.003" length="0.045"/>
+            </geometry>
+        </collision>
+        <collision>
+            <origin xyz="0.05 -0.035 -0.07" rpy="0 -1.0 0"/>
+            <geometry>
+                <cylinder radius="0.003" length="0.045"/>
             </geometry>
         </collision>
