Commit message: Creation of frea_motion_control package
Updated READMEs, and created the base_link_tf_publisher node, to calculate the transform from the base_link to the chassis_link

File: frea_description/urdf/chassis/chassis.urdf.xacro (robot description, xacro)
@@ -16,5 +16,5 @@
         <limit effort="0" velocity="0"/>
         <origin xyz="0 0 0" rpy="0 ${-30*3.14/180} 0"/>
-        <parent link="base_link"/>
+        <parent link="fixed_base_link"/>
         <child link="chassis_link"/>
     </joint>

File: frea_description/urdf/frea.urdf.xacro (robot description, xacro)
@@ -12,5 +12,5 @@
      links without mass properties - thus the base_link must have mass and
      cannot be the "parent" link -->
-<link name="base_link">
+<link name="fixed_base_link">
     <inertial>
         <mass value="1e-3"/>
@@ -21,5 +21,5 @@
 <joint name="parent_joint" type="fixed">
     <parent link="parent_link"/>
-    <child link="base_link"/>
+    <child link="fixed_base_link"/>
 </joint>
 <gazebo>

Commit message: Visualising the DART simulation now works.
Scaled the stl files to the correct size, and updated urdf files accordingly. I ahve also implemented the ROS control section of frea_dart, and updated controller naming conventions accordingly. Unfortunately frea_dart seems to crash during collision detection (in World::step->ConstraintSolver::solve()->FCLCollisionDetector::collide()...) due to a segmentation fault. Not certain what I've forgotten to initialise, but I suppose we'll work it out eventually.

File: frea_description/urdf/chassis/chassis.urdf.xacro (robot description, xacro)
@@ -29,6 +29,5 @@
             <origin xyz="0 0 0" rpy="${30*3.14/180} 0 1.57"/>
             <geometry>
-                <mesh filename="$(find frea_description)/meshes/chassis.stl"
-                      scale="0.001 0.001 0.001"/>
+                <mesh filename="$(find frea_description)/meshes/chassis.stl"/>
             </geometry>
         </visual>

File: frea_description/urdf/chassis/wheel/wheel.urdf.xacro (robot description, xacro)
@@ -21,6 +21,5 @@
             <origin xyz="0 ${-mirror*0.021} 0" rpy="0 0 0"/>
             <geometry>
-                <mesh filename="$(find frea_description)/meshes/wheel.stl"
-                      scale="0.001 ${mirror*0.001} 0.001"/>
+                <mesh filename="$(find frea_description)/meshes/wheel.stl"/>
             </geometry>
         </visual>

File: frea_description/urdf/dart/frea_dart.urdf.xacro (robot description, xacro)
@@ -21,3 +21,2 @@
 </joint>
 </robot>
-</robot>

File: frea_description/urdf/head/ears/left_ear.urdf.xacro (robot description, xacro)
@@ -21,6 +21,5 @@
            <origin xyz="0 0.0025 0" rpy="1.57 -1.57 0"/>
            <geometry>
-                <mesh filename="$(find frea_description)/meshes/left_ear.stl"
-                      scale="0.001 0.001 0.001"/>
+                <mesh filename="$(find frea_description)/meshes/left_ear.stl"/>
             </geometry>
         </visual>

File: frea_description/urdf/head/ears/right_ear.urdf.xacro (robot description, xacro)
@@ -21,6 +21,5 @@
            <origin xyz="0 0.0025 0" rpy="-1.57 -1.57 0"/>
            <geometry>
-                <mesh filename="$(find frea_description)/meshes/right_ear.stl"
-                      scale="0.001 0.001 0.001"/>
+                <mesh filename="$(find frea_description)/meshes/right_ear.stl"/>
             </geometry>
         </visual>

File: frea_description/urdf/head/head.urdf.xacro (robot description, xacro)
@@ -32,6 +32,5 @@
             <origin xyz="0 0 0" rpy="0 0 1.57"/>
             <geometry>
-                <mesh filename="$(find frea_description)/meshes/head.stl"
-                      scale="0.001 0.001 0.001"/>
+                <mesh filename="$(find frea_description)/meshes/head.stl"/>
             </geometry>
         </visual>

File: frea_description/urdf/head/mouth/mouth.urdf.xacro (robot description, xacro)
@@ -22,6 +22,5 @@
             <origin xyz="0.0785 0 -0.0075" rpy="0 0 1.57"/>
             <geometry>
-                <mesh filename="$(find frea_description)/meshes/mouth.stl"
-                      scale="0.001 0.001 0.001"/>
+                <mesh filename="$(find frea_description)/meshes/mouth.stl"/>
             </geometry>
         </visual>

File: frea_description/urdf/neck/neck_end.urdf.xacro (robot description, xacro)
@@ -21,6 +21,5 @@
             <origin xyz="0 0 0" rpy="1.57 0 1.57"/>
             <geometry>
-                <mesh filename="$(find frea_description)/meshes/end_link.stl"
-                      scale="0.001 0.001 0.001"/>
+                <mesh filename="$(find frea_description)/meshes/end_link.stl"/>
             </geometry>
         </visual>

File: frea_description/urdf/neck/neck_mid.urdf.xacro (robot description, xacro)
@@ -21,6 +21,5 @@
             <origin xyz="0 0 0" rpy="1.57 0 1.57"/>
             <geometry>
-                <mesh filename="$(find frea_description)/meshes/mid_link.stl"
-                      scale="0.001 0.001 0.001"/>
+                <mesh filename="$(find frea_description)/meshes/mid_link.stl"/>
             </geometry>
         </visual>
