Commit message: DART Does not crash!
DART now doesn't crash due to explosive controller responses. This was in part due to poorly tuned controllers and in part due to a 0.01 timestep. Changing to 0.001 fixed this. In addition, I've updated/fixed some issues with the URDF.

File: frea_description/urdf/dart/frea_dart.urdf.xacro (robot description, xacro)
@@ -1,10 +1,4 @@
 <?xml version="1.0"?>
 <robot xmlns:xacro="http://www.ros.org/wiki/xacro">
-<!-- World link for dart -->
-<link name="world"/>
-<joint name="world_frea" type="floating">
-    <parent link="world"/>
-    <child link="parent_link"/>
-</joint>
 <!-- Extra head and tail links for adjustable weight -->
 <link name="head_weight_link"/>

File: frea_description/urdf/sensors/imu.urdf.xacro (robot description, xacro)
@@ -2,5 +2,5 @@
 <robot xmlns:xacro="http://www.ros.org/wiki/xacro">
 <xacro:macro name="imu" params="parent name xyz">
-    <joint name="${name}_imu_sensor" type="fixed">
+    <joint name="${name}_sensor" type="fixed">
         <origin xyz="${xyz}" rpy="0 0 0"/>
         <parent link="${parent}"/>
