Commit message: minor urdf fix

File: frea_description/urdf/chassis/wheel/wheel.urdf.xacro (robot description, xacro)
@@ -19,5 +19,5 @@
         </inertial>
         <visual>
-            <origin xyz="0 ${-mirror*0.021} 0" rpy="0 0 0"/>
+            <origin xyz="0 -0.021 0" rpy="0 0 0"/>
             <geometry>
                 <mesh filename="$(find frea_description)/meshes/wheel.stl"/>
